File: ESP12-Break-02.sch (KiCad schematic (older format))
At the start: 21 parts, among them J1 CONN_01X08, J2 CONN_01X08, J3 GS2, SW1 Switch, SW2 Switch, U1 ESP-12, U2 AP2112K-3.3TRG1

Commit message: Change value on Neopixel Capacitor
Parts:
- C4: value 1uF -> 0.1uF
Connections:
- net labels added: GPIO
- wire segments 72 -> 77
- no-connect marks 2 -> 1
Other:
- note added: "DEEP SLEEP"
- note added: "NEOPIXEL"
- note added: "RESET"
- note added: "USER/PROG"
- moved on the sheet: U2

Commit message: Minor changes
Connections:
- wire segments 77 -> 85
Changed lines of the file:
@@
 	-1   0    0    1
 $EndComp
-Text Label 9775 4275 2    60   ~ 0
+Text Label 9650 4175 2    60   ~ 0
 GPIO15
 Text Label 3225 4550 0    60   ~ 0
 RESET
-Text Label 9175 2150 2    60   ~ 0
-GND
-Text Label 9775 4675 2    60   ~ 0
+Text Label 10000 4725 0    60   ~ 0
 RESET
 $Comp
@@
 	1    0    0    -1
 $EndComp
-Text Label 9800 2050 2    60   ~ 0
-GND
-Text Label 7925 2050 2    60   ~ 0
-GND
 $Comp
 L power:PWR_FLAG #FLG02
@@
 	1    0    0    -1
 $EndComp
-Text Label 10250 2050 2    60   ~ 0
+Text Label 9175 2425 2    60   ~ 0
 GND
 Text Label 10250 1425 0    60   ~ 0
@@
 	8875 2050 8875 1725
 Wire Wire Line
-	9175 2025 9175 2150
-Wire Wire Line
-	9800 1975 9800 2050
-Wire Wire Line
-	7925 1975 7925 2050
-Wire Wire Line
 	6675 1175 6675 1275
 Wire Wire Line
@@
 Wire Wire Line
 	10250 1425 10250 1625
-Wire Wire Line
-	10250 1975 10250 2050
 Connection ~ 10250 1625
 Wire Wire Line
@@
 Text Notes 6175 4150 0    60   ~ 0
 NEOPIXEL
-Text Notes 9450 4100 0    60   ~ 0
+Text Notes 9475 3850 0    60   ~ 0
 DEEP SLEEP
 Wire Notes Line
 	6300 450  6300 3350
+Wire Wire Line
+	9775 4275 9775 4175
+Wire Wire Line
+	9775 4175 9650 4175
+Wire Wire Line
+	9775 4675 9775 4725
+Wire Wire Line
+	9775 4725 10000 4725
+Wire Wire Line
+	7925 2225 9175 2225
+Wire Wire Line
+	7925 1975 7925 2225
+Wire Wire Line
+	10250 1975 10250 2225
+Wire Wire Line
+	9800 1975 9800 2225
+Connection ~ 9800 2225
+Wire Wire Line
+	9800 2225 10250 2225
+Wire Wire Line
+	9175 2025 9175 2225
+Connection ~ 9175 2225
+Wire Wire Line
+	9175 2225 9800 2225
+Wire Wire Line
+	9175 2425 9175 2225
 $EndSCHEMATC
