File: Breakout/ESP12-Break-02.sch (KiCad schematic (older format))
At the start: 21 parts, among them J1 CONN_01X08, J2 CONN_01X08, J3 GS2, SW1 Switch, SW2 Switch, U1 ESP-12, U2 AP2112K-3.3TRG1

Commit message: Reorganize & add USB version
Parts:
- renumbered SW1 to RESET1, SW2 to USER/PROG1
Other:
- note removed: "RESET"
- note removed: "USER/PROG"
Changed lines of the file:
@@
 BUTTONS & LEDS
 $Comp
-L icezum:Switch SW1
+L icezum:Switch RESET1
 U 1 1 5A90CF8A
 P 2625 4550
-F 0 "SW1" H 2925 4775 60  0000 L BNN
+F 0 "RESET1" H 2875 4800 60  0000 L BNN
 F 1 "Switch" H 2850 4375 60  0000 L BNN
 F 2 "OSHwi:SW_SPST_B3U-1000P" H 2625 4550 60  0001 C CNN
@@
 L wickerlib:DIODE-GEN-PURP-75V-250MA-1N4148WTR-SOD123 D2
 U 1 1 5A917918
-P 8675 2675
-F 0 "D2" V 8800 2675 50  0000 L CNN
-F 1 "1N4148" V 8550 2550 50  0000 L CNN
-F 2 "OSHwi:D_SOD-123" H 8675 2325 50  0001 C CIN
-F 3 "http://www.vishay.com/docs/85752/bas16ws.pdf" V 8675 2700 5   0001 C CNN
-F 4 "DIODE GEN PURP 75V 250MA 1N4148 SOD123" H 8675 2325 50  0001 C CIN "Description"
-F 5 "SMC Diode" H 8675 2325 50  0001 C CIN "MF_Name"
-F 6 "1N4148WTR" H 8675 2325 50  0001 C CIN "MF_PN"
-F 7 "Digikey" H 8675 2325 50  0001 C CIN "S1_Name"
-F 8 "1655-1360-1-ND" H 8675 2325 50  0001 C CIN "S1_PN"
-	1    8675 2675
+P 8600 2950
+F 0 "D2" V 8725 2950 50  0000 L CNN
+F 1 "1N4148" V 8475 2825 50  0000 L CNN
+F 2 "OSHwi:D_SOD-123" H 8600 2600 50  0001 C CIN
+F 3 "http://www.vishay.com/docs/85752/bas16ws.pdf" V 8600 2975 5   0001 C CNN
+F 4 "DIODE GEN PURP 75V 250MA 1N4148 SOD123" H 8600 2600 50  0001 C CIN "Description"
+F 5 "SMC Diode" H 8600 2600 50  0001 C CIN "MF_Name"
+F 6 "1N4148WTR" H 8600 2600 50  0001 C CIN "MF_PN"
+F 7 "Digikey" H 8600 2600 50  0001 C CIN "S1_Name"
+F 8 "1655-1360-1-ND" H 8600 2600 50  0001 C CIN "S1_PN"
+	1    8600 2950
 	0    -1   -1   0
 $EndComp
-Text Label 8925 2675 0    60   ~ 0
+Text Label 8850 2950 0    60   ~ 0
 RESET
-Text Label 8375 2675 2    60   ~ 0
+Text Label 8300 2950 2    60   ~ 0
 RESET_5V
 $Comp
 L wickerlib:DIODE-GEN-PURP-75V-250MA-1N4148WTR-SOD123 D3
 U 1 1 5A9185CE
-P 10025 2675
-F 0 "D3" V 10150 2675 50  0000 L CNN
-F 1 "1N4148" V 9900 2550 50  0000 L CNN
-F 2 "OSHwi:D_SOD-123" H 10025 2325 50  0001 C CIN
-F 3 "http://www.vishay.com/docs/85752/bas16ws.pdf" V 10025 2700 5   0001 C CNN
-F 4 "DIODE GEN PURP 75V 250MA 1N4148 SOD123" H 10025 2325 50  0001 C CIN "Description"
-F 5 "SMC Diode" H 10025 2325 50  0001 C CIN "MF_Name"
-F 6 "1N4148WTR" H 10025 2325 50  0001 C CIN "MF_PN"
-F 7 "Digikey" H 10025 2325 50  0001 C CIN "S1_Name"
-F 8 "1655-1360-1-ND" H 10025 2325 50  0001 C CIN "S1_PN"
-	1    10025 2675
+P 9950 2950
+F 0 "D3" V 10075 2950 50  0000 L CNN
+F 1 "1N4148" V 9825 2825 50  0000 L CNN
+F 2 "OSHwi:D_SOD-123" H 9950 2600 50  0001 C CIN
+F 3 "http://www.vishay.com/docs/85752/bas16ws.pdf" V 9950 2975 5   0001 C CNN
+F 4 "DIODE GEN PURP 75V 250MA 1N4148 SOD123" H 9950 2600 50  0001 C CIN "Description"
+F 5 "SMC Diode" H 9950 2600 50  0001 C CIN "MF_Name"
+F 6 "1N4148WTR" H 9950 2600 50  0001 C CIN "MF_PN"
+F 7 "Digikey" H 9950 2600 50  0001 C CIN "S1_Name"
+F 8 "1655-1360-1-ND" H 9950 2600 50  0001 C CIN "S1_PN"
+	1    9950 2950
 	0    -1   -1   0
 $EndComp
-Text Label 10275 2675 0    60   ~ 0
+Text Label 10200 2950 0    60   ~ 0
 RXD
-Text Label 9725 2675 2    60   ~ 0
+Text Label 9650 2950 2    60   ~ 0
 RXD_5V
 $Comp
@@
 	9800 1625 9800 1675
 Wire Wire Line
-	8800 2675 8925 2675
-Wire Wire Line
-	8500 2675 8375 2675
-Wire Wire Line
-	10150 2675 10275 2675
-Wire Wire Line
-	9850 2675 9725 2675
+	8725 2950 8850 2950
+Wire Wire Line
+	8425 2950 8300 2950
+Wire Wire Line
+	10075 2950 10200 2950
+Wire Wire Line
+	9775 2950 9650 2950
 Wire Wire Line
 	5875 4525 5200 4525
@@
 Wire Wire Line
 	2925 4550 2625 4550
-Text Notes 2075 4175 0    60   ~ 0
-RESET
 $Comp
 L device:R R2
@@
 GPIO
 $Comp
-L icezum:Switch SW2
+L icezum:Switch USER/PROG1
 U 1 1 5A9260B4
 P 2650 5600
-F 0 "SW2" H 2950 5825 60  0000 L BNN
+F 0 "USER/PROG1" H 2775 5800 60  0000 L BNN
 F 1 "Switch" H 2875 5425 60  0000 L BNN
 F 2 "OSHwi:SW_SPST_B3U-1000P" H 2650 5600 60  0001 C CNN
@@
 Wire Wire Line
 	2950 5600 2650 5600
-Text Notes 1950 5225 0    60   ~ 0
-USER/PROG
 Connection ~ 5200 4525
 Wire Wire Line
